Commit message: ADD Ardupilot gazebo physics simulator

File: bluerov2_description/urdf/actuators.xacro (robot description, xacro)
@@ -8,32 +8,60 @@
     aware that Gazebo does not use the SNAME convention per default.
   -->
-  <!-- IMPROVE -->
+  <!-- Thrusters for SITL to apply forces to -->
+  <!-- Courtesy of NYUAD Robosub https://github.com/nyuad-robosub/bluerov2/tree/5ecac19e27db1d43a663141c8704355a17c1abf3 -->
+  <xacro:macro name="thruster_sitl_macro" params="robot_namespace thruster_id *origin">
+    <link name="${robot_namespace}/thruster_sitl_${thruster_id}">
+      <inertial>
+        <origin xyz="0 0 0" rpy="0 0 0"/>
+        <mass value="0.0001"/>
+        <inertia ixx="0.00000002" ixy="0.0" ixz="0.0" iyy="0.00000002" iyz="0.0" izz="0.00000002"/>
+      </inertial>
+    </link>
+     <joint name="${robot_namespace}/thruster_sitl_${thruster_id}_joint" type="revolute">
+      <xacro:insert_block name="origin" />
+      <axis xyz="1 0 0" />
+      <limit effort="0.0" upper="0.0" lower="0.0" velocity="0.0"/>
+      <parent link="${robot_namespace}/base_link" />
+      <child link="${robot_namespace}/thruster_sitl_${thruster_id}" />
+    </joint>
+    <gazebo reference="${robot_namespace}/thruster_sitl_${thruster_id}">
+      <selfCollide>false</selfCollide>
+    </gazebo>
+  </xacro:macro>
   <xacro:thruster_macro robot_namespace="${namespace}" thruster_id="0">
     <origin xyz="0.1355 -0.1 -0.0725" rpy="0 0 0.7853981634"/>
   </xacro:thruster_macro>
-  <!-- IMPROVE -->
+  <xacro:thruster_sitl_macro robot_namespace="${namespace}" thruster_id="0">
+    <origin xyz="0.1355 -0.1 -0.0725" rpy="1.5707963 1.5707963 -0.78539815"/>
+  </xacro:thruster_sitl_macro>
   <xacro:thruster_macro robot_namespace="${namespace}" thruster_id="1">
     <origin xyz="0.1355 0.1 -0.0725" rpy="0 0 -0.7853981634"/>
   </xacro:thruster_macro>
-  <!-- IMPROVE -->
+  <xacro:thruster_sitl_macro robot_namespace="${namespace}" thruster_id="1">
+    <origin xyz="0.1355 0.1 -0.0725" rpy="1.5707963 1.5707963 3.92699075"/>
+  </xacro:thruster_sitl_macro>
   <xacro:thruster_macro robot_namespace="${namespace}" thruster_id="2">
     <origin xyz="-0.1475 -0.1 -0.0725" rpy="0 0 2.3561944902"/>
   </xacro:thruster_macro>
-  <!-- IMPROVE -->
+  <xacro:thruster_sitl_macro robot_namespace="${namespace}" thruster_id="2">
+    <origin xyz="-0.1475 -0.1 -0.0725" rpy="1.5707963 1.5707963 0.78540075"/>
+  </xacro:thruster_sitl_macro>
   <xacro:thruster_macro robot_namespace="${namespace}" thruster_id="3">
     <origin xyz="-0.1475 0.1 -0.0725" rpy="0 0 -2.3561944902"/>
   </xacro:thruster_macro>
-  <!-- IMPROVE -->
+  <xacro:thruster_sitl_macro robot_namespace="${namespace}" thruster_id="3">
+    <origin xyz="-0.1475 0.1 -0.0725" rpy="1.5707963 1.5707963 2.35619445"/>
+  </xacro:thruster_sitl_macro>
   <xacro:thruster_macro robot_namespace="${namespace}" thruster_id="4">
     <origin xyz="0.0025 -0.1105 -0.005" rpy="0 -1.5707963268 0"/>
   </xacro:thruster_macro>
-  <!-- IMPROVE -->
+  <xacro:thruster_sitl_macro robot_namespace="${namespace}" thruster_id="4">
+    <origin xyz="0.0025 -0.1105 -0.005" rpy="3.1415926 0 0"/>
+  </xacro:thruster_sitl_macro>
   <xacro:thruster_macro robot_namespace="${namespace}" thruster_id="5">
     <origin xyz="0.0025 0.1105 -0.005" rpy="0 -1.5707963268 0"/>
   </xacro:thruster_macro>
-  <!-- ###### TO BE IMPLEMENTED ###### -->
-  <!-- Mount a Beacon actuator -->
-  <!-- <xacro:default_beacon namespace="${namespace}" parent_link="${namespace}/base_link">
-    <origin xyz="0 0 0" rpy="0 0 0"/>
-  </xacro:default_beacon> -->
+  <xacro:thruster_sitl_macro robot_namespace="${namespace}" thruster_id="5">
+    <origin xyz="0.0025 0.1105 -0.005" rpy="3.1415926 0 0"/>
+  </xacro:thruster_sitl_macro>
 </robot>

File: bluerov2_description/urdf/base.xacro (robot description, xacro)
@@ -81,4 +81,10 @@
     <gazebo reference="${namespace}/base_link">
       <selfCollide>false</selfCollide>
+      <!-- IMU SITL SENSOR -->
+      <sensor type="imu" name="imu_sensor">
+        <pose>0 0 0 0 0 0</pose>
+        <always_on>true</always_on>
+        <update_rate>1000.0</update_rate>
+      </sensor>
     </gazebo>
     <!-- Set up hydrodynamic plugin given as input parameter -->
@@ -88,4 +94,6 @@
     <!-- Include the sensor modules: 3D Pose, IMU, Pressure, Camera -->
     <xacro:include filename="$(find bluerov2_description)/urdf/sensors.xacro"/>
+    <!-- Include Ardusub SITL, this will apply forces and torques to the vehicle based on the delta x from sim_vehicle.py -->
+    <xacro:include filename="$(find bluerov2_description)/urdf/sitl.xacro"/>
   </xacro:macro>
 </robot>
