Commit message: Add sonars and Ping2 to URDF

File: bluerov2_description/urdf/base.xacro (robot description, xacro)
@@ -7,4 +7,6 @@
   <!-- Loading vehicle's specific macros -->
   <xacro:include filename="$(find bluerov2_description)/urdf/snippets.xacro"/>
+  <!-- Loading sonar macros -->
+  <xacro:include filename="$(find sonar_testing)/model/sonars.urdf.xacro"/>
   <!-- ADDED  -->
   <xacro:include filename="$(find uuv_gazebo_ros_plugins)/urdf/snippets.xacro"/>

File: bluerov2_description/urdf/sensors.xacro (robot description, xacro)
@@ -26,3 +26,16 @@
   <!-- Mount a GPS. -->
   <xacro:default_gps namespace="${namespace}" parent_link="${namespace}/base_link" />
+  <!-- Mount the sonars -->
+	<xacro:ping360_macro parent_link="${namespace}/base_link" prefix="${namespace}/" namespace="/bluerov2">
+		<origin xyz="0.15 0.1 0.1" rpy="0 0 0"/>
+		<axis xyz="0 0 1"/>
+	</xacro:ping360_macro>
+	<xacro:mbe_macro parent_link="${namespace}/base_link" prefix="${namespace}/" namespace="/bluerov2">
+    <origin xyz="0.15 -0.1 0.1" rpy="0 0.174533 0"/>
+    <axis xyz="0 0 1"/>
+	</xacro:mbe_macro>
+	<xacro:ping2_macro parent_link="${namespace}/base_link" prefix="${namespace}/" namespace="/bluerov2">
+    <origin xyz="0 0.2 0.05" rpy="0 1.57079632679 0" />
+    <axis xyz="0 0 1" />
+	</xacro:ping2_macro>
 </robot>
