Commit message: ADD heavy config sonar sensors

File: bluerov2_description_heavy/urdf/base.xacro (robot description, xacro)
@@ -8,5 +8,5 @@
   <xacro:include filename="$(find bluerov2_description)/urdf/snippets.xacro"/>
   <!-- Loading sonar macros -->
-  <!-- <xacro:include filename="$(find sonar_testing)/models/sonars.urdf.xacro"/> -->
+  <xacro:include filename="$(find sonar_testing)/models/sonars.urdf.xacro"/>
   <!-- ADDED  -->
   <xacro:include filename="$(find uuv_gazebo_ros_plugins)/urdf/snippets.xacro"/>

File: bluerov2_description_heavy/urdf/sensors.xacro (robot description, xacro)
@@ -27,10 +27,10 @@
   <xacro:default_gps namespace="${namespace}" parent_link="${namespace}/base_link" />
   <!-- Mount the sonars -->
-	<!-- <xacro:ping360_macro parent_link="${namespace}/base_link" prefix="${namespace}/" namespace="/bluerov2">
-		<origin xyz="0.15 0.1 0.1" rpy="0 0 0"/>
+	<xacro:ping360_macro parent_link="${namespace}/base_link" prefix="${namespace}/" namespace="/bluerov2">
+		<origin xyz="0.15 0.1 0.16" rpy="0 0 0"/>
 		<axis xyz="0 0 1"/>
 	</xacro:ping360_macro>
 	<xacro:mbe_macro parent_link="${namespace}/base_link" prefix="${namespace}/" namespace="/bluerov2">
-    <origin xyz="0.15 -0.1 0.1" rpy="0 0.174533 0"/>
+    <origin xyz="0.15 -0.1 0.16" rpy="0 0.174533 0"/>
     <axis xyz="0 0 1"/>
 	</xacro:mbe_macro>
@@ -38,4 +38,4 @@
     <origin xyz="0 0.2 0.05" rpy="0 1.57079632679 0" />
     <axis xyz="0 0 1" />
-	</xacro:ping2_macro> -->
+	</xacro:ping2_macro>
 </robot>
